Commit message: XACRO cleanup

File: tracer_description/models/xacro/tracer_wheels.xacro (robot description, xacro)
@@ -26,5 +26,5 @@
             <xacro:insert_block name="origin" />
             <axis xyz="0 1 0" rpy="0 0 0" />
-            <limit lower="-1.79769e+308" upper="1.79769e+308" effort="20.0" velocity="5.0"/>
+            <limit lower="-1.79769e+308" upper="1.79769e+308" effort="20.0" velocity="5.0" />
         </joint>
     </xacro:macro>
