Commit message: XACRO cleanup

File: tracer_description/models/xacro/tracer_castor_wheels.xacro (robot description, xacro)
@@ -22,5 +22,5 @@
             <parent link="${name}_castor_link" />
             <child link="${name}_wheel_link"/>
-            <dynamics damping="0.0" friction="0.0" />
+            <dynamics damping="0.2" friction="0.2" />
             <xacro:insert_block name="origin" />
             <axis xyz="0 0 1" rpy="0 0 0" />
